Commit message: Full design review: CG-aware gait, tibia knee-neck strength fix, checkers, docs, issues
Findings from the 2026-09-04 whole-repo review (systems / mechanical / docs):

Gait (S-01/S-02): the stability margin assumed the CG at the body origin, but the
URDF mass model puts it at y=-39mm (Cabin). polygon_margin now uses config.CG_XY;
the neutral foot pattern is shifted rearward (STANCE_OFF_XY -30), rear-leg SWAY
raised to 40mm, BODY_H_MIN 105->110, LIM_YAW_POD 22->30 (mesh contact starts at
34deg). Worst-case margin -23.7 -> +10.9mm, IK failures 0. sim_gait [3] now sweeps
all commands/phases with 3/4-point static leg loads: worst hip torque 18.5 kgf.cm
(was a single-point 8.9). FOOT_GROUND_OFFSET recalibrated 18.6->20.98
(TIBIA_LEN 155.98, D_KNEE 210.2/119.1).

Mechanical (M-01/M-02): the tibia knee neck was cut to 11mm^2 by symmetric 45deg
wedges (SF ~0.1). Replaced by an exact swept-femur subtraction (_femur_knee_sweep)
plus a 3mm outer doubler -> 115mm^2, SF 2.1. New tools/check_leg_link_strength.py
(section-stress scan, SF>=2). HORN_PILOT_D 2.0->2.2 for the M2.6 horn screws.

Tooling/docs: make_plates registers 14 STLs / 6 plates (+PLA_Matte_Blue_5_HeadTop
for PR-08, rot_x90 rule); regenerated Tibia/Gray/White plates; manifest tallies
fixed; README/HANDOFF/assembly/wiring/BOM updated (gate load 1.2kg x 155mm lever,
UBEC 10A vs 9-14A, cable-hole test, claw epoxy, camera jig, tapping notes).
Physics metrics regenerated with the new gait (roll 6.4 -> 3.2deg, no fall).

Issues: 4 new (EL-09 UBEC rating, EL-10 idle heat, L-11 hip-torque decision,
I-08 sim_physics saturation), 19 bodies updated, build_plan regenerated.

Co-Authored-By: Claude Fable 5.1 <noreply@anthropic.com>

File: hardware/urdf/tachikoma.urdf (robot description, URDF)
Before this commit: robot tachikoma, 23 links, 22 joints
Links:
- link leg_fl_coxa: mass 0.091059341 -> 0.091047964
- link leg_fl_femur: mass 0.095793916 -> 0.095788395
- link leg_fl_tibia: mass 0.087444704 -> 0.089251573
- link leg_fr_coxa: mass 0.091059341 -> 0.091047964
- link leg_fr_femur: mass 0.095793916 -> 0.095788395
- link leg_fr_tibia: mass 0.087444704 -> 0.089251573
- link leg_rl_coxa: mass 0.091059341 -> 0.091047964
- link leg_rl_femur: mass 0.095793916 -> 0.095788395
- link leg_rl_tibia: mass 0.087444704 -> 0.089251573
- link leg_rr_coxa: mass 0.091059341 -> 0.091047964
- link leg_rr_femur: mass 0.095793916 -> 0.095788395
- link leg_rr_tibia: mass 0.087444704 -> 0.089251573
