Commit message: 実機設計を再監査し、制御・内部形状・検証基盤の不具合を修正する
開始時515ファイルを用途別に点検し、全STL/URDFを再生成。
実制御を含む89条件の物理計算と18姿勢の干渉検査を保存した。
最終23検査は14合格・8不合格・1未検証。頭部収納、支持、脚装飾、
TPU足裏などの未解決事項を残し、実機の組立・歩行合格とは扱わない。

元モデル・既存3MF・旧画像動画を保持。内部形状10 STLと配置2 STLを
更新し、製作への影響・不採用候補・再現条件を監査報告に記録した。
メーカー原本コピーと再生成できる衝突キャッシュはGitに含めない。

検証: 生成3工程、回帰53件、物理回帰16件、firmwareホスト試験、
通常/校正ビルド。工程別ログと入力SHAをdocs/auditsへ保存。

Refs #80, #85, #81, #82, #83, #84, #93, #78

File: hardware/urdf/tachikoma.urdf (robot description, URDF)
Before this commit: robot tachikoma, 23 links, 22 joints
Links:
- link arm_l_forearm: mass 0.010796046 -> 0.008528994
- link arm_l_shoulder: mass 0.023752007 -> 0.023542634
- link arm_l_upper: mass 0.036488675 -> 0.036488674
- link arm_r_forearm: mass 0.010796046 -> 0.008528994
- link arm_r_shoulder: mass 0.023752007 -> 0.023542634
- link arm_r_upper: mass 0.036488675 -> 0.036488674
- link base_link: mass 1.516523023 -> 1.466825865
- link leg_fl_coxa: mass 0.091047964 -> 0.083787095
- link leg_fl_tibia: mass 0.089251573 -> 0.094299363; geometry collision mesh filename=meshes/leg_fl_tibia__col_0.stl; visual mesh filename=meshes/leg_fl_tibia__vis_333333.stl
- link leg_fr_coxa: mass 0.091047964 -> 0.083787095
- link leg_fr_tibia: mass 0.089251573 -> 0.094299363; geometry collision mesh filename=meshes/leg_fr_tibia__col_0.stl; visual mesh filename=meshes/leg_fr_tibia__vis_333333.stl
- link leg_rl_coxa: mass 0.091047964 -> 0.083787095
- link leg_rl_tibia: mass 0.089251573 -> 0.094299363; geometry collision mesh filename=meshes/leg_rl_tibia__col_0.stl; visual mesh filename=meshes/leg_rl_tibia__vis_333333.stl
- link leg_rr_coxa: mass 0.091047964 -> 0.083787095
- link leg_rr_tibia: mass 0.089251573 -> 0.094299363; geometry collision mesh filename=meshes/leg_rr_tibia__col_0.stl; visual mesh filename=meshes/leg_rr_tibia__vis_333333.stl
Joints:
- joint arm_l_elbow: limit lower=0.000000 upper=1.658063 effort=0.22 velocity=13.0 -> lower=0.000000 upper=1.658063 effort=0.2026707666666667 velocity=13.08996938995747
- joint arm_l_pitch: limit lower=-0.785398 upper=1.483530 effort=0.22 velocity=13.0 -> lower=-0.785398 upper=1.483530 effort=0.2026707666666667 velocity=13.08996938995747
- joint arm_l_yaw: limit lower=-0.261799 upper=0.261799 effort=0.22 velocity=13.0 -> lower=-0.261799 upper=0.261799 effort=0.2026707666666667 velocity=13.08996938995747
- joint arm_r_elbow: limit lower=0.000000 upper=1.658063 effort=0.22 velocity=13.0 -> lower=0.000000 upper=1.658063 effort=0.2026707666666667 velocity=13.08996938995747
- joint arm_r_pitch: limit lower=-0.785398 upper=1.483530 effort=0.22 velocity=13.0 -> lower=-0.785398 upper=1.483530 effort=0.2026707666666667 velocity=13.08996938995747
- joint arm_r_yaw: limit lower=-0.261799 upper=0.261799 effort=0.22 velocity=13.0 -> lower=-0.261799 upper=0.261799 effort=0.2026707666666667 velocity=13.08996938995747
- joint leg_fl_knee: limit lower=-0.767945 upper=0.767945 effort=1.96 velocity=6.5 -> lower=-0.767945 upper=0.767945 effort=1.955881861111111 velocity=7.033416388633864
- joint leg_fl_pitch: limit lower=-0.785398 upper=0.959931 effort=1.96 velocity=6.5 -> lower=-0.785398 upper=0.959931 effort=1.955881861111111 velocity=7.033416388633864
- joint leg_fl_yaw: limit lower=-0.698132 upper=0.698132 effort=1.96 velocity=6.5 -> lower=-0.698132 upper=0.698132 effort=1.955881861111111 velocity=7.033416388633864
- joint leg_fr_knee: limit lower=-0.767945 upper=0.767945 effort=1.96 velocity=6.5 -> lower=-0.767945 upper=0.767945 effort=1.955881861111111 velocity=7.033416388633864
- joint leg_fr_pitch: limit lower=-0.785398 upper=0.959931 effort=1.96 velocity=6.5 -> lower=-0.785398 upper=0.959931 effort=1.955881861111111 velocity=7.033416388633864
- joint leg_fr_yaw: limit lower=-0.698132 upper=0.698132 effort=1.96 velocity=6.5 -> lower=-0.698132 upper=0.698132 effort=1.955881861111111 velocity=7.033416388633864
- joint leg_rl_knee: limit lower=-0.767945 upper=0.767945 effort=1.96 velocity=6.5 -> lower=-0.767945 upper=0.767945 effort=1.955881861111111 velocity=7.033416388633864
- joint leg_rl_pitch: limit lower=-0.785398 upper=0.959931 effort=1.96 velocity=6.5 -> lower=-0.785398 upper=0.959931 effort=1.955881861111111 velocity=7.033416388633864
- joint leg_rl_yaw: limit lower=-0.698132 upper=0.698132 effort=1.96 velocity=6.5 -> lower=-0.698132 upper=0.698132 effort=1.955881861111111 velocity=7.033416388633864
- joint leg_rr_knee: limit lower=-0.767945 upper=0.767945 effort=1.96 velocity=6.5 -> lower=-0.767945 upper=0.767945 effort=1.955881861111111 velocity=7.033416388633864
- joint leg_rr_pitch: limit lower=-0.785398 upper=0.959931 effort=1.96 velocity=6.5 -> lower=-0.785398 upper=0.959931 effort=1.955881861111111 velocity=7.033416388633864
- joint leg_rr_yaw: limit lower=-0.698132 upper=0.698132 effort=1.96 velocity=6.5 -> lower=-0.698132 upper=0.698132 effort=1.955881861111111 velocity=7.033416388633864
